Commit message: update limits to valuese that match robot visualization

File: robot/robot.urdf (robot description, URDF)
Before this commit: robot 6dof_robot_arm, 0 links, 6 joints
Joints:
- joint joint1: limit lower=-110 upper=20 -> lower=-180 upper=180
- joint joint2: limit lower=-180 upper=180 -> lower=-60 upper=60
- joint joint3: limit lower=-180 upper=180 -> lower=-120 upper=120
- joint joint4: limit lower=-130 upper=120 -> lower=-180 upper=180
- joint joint5: limit lower=-180 upper=180 -> lower=-90 upper=90
- joint joint6: limit lower=-20 upper=40 -> lower=-180 upper=180
